File: PFC.kicad_sch (KiCad schematic)
At the start: 42 parts, among them IC1 UCC28180D, J1 Conn_01x02_Pin, J2 Conn_01x02_Pin, J3 Conn_01x04_Pin, J4 Conn_01x02_Pin, Q1 IMBG120R234M2HXTMA1, Q2 T2N7002AK, Q3 T2N7002AK, U1 MGJ2D241505SC, U2 MGJ2D241505SC, U3 UCC21520DW, U4 L7805, U5 MCP6002-xSN, U6 MCP6567, U7 74AHC1G14, U8 EL817

Commit message: initial work
Parts:
- removed C1, C2: C, symbol Device:C
- removed D1, D2: IDWD30G120C5, Package_TO_SOT_THT:TO-247-2_Horizontal_TabDown, symbol Diode:C4D20120H
- removed D3: BZV55B16, Diode_SMD:D_MiniMELF, symbol Diode:BZV55B16
- removed D4: BAT54C, Package_TO_SOT_SMD:SOT-23, symbol Diode:BAT54C
- removed IC1: UCC28180D, Package_SO:SOIC-8_3.9x4.9mm_P1.27mm, symbol New_Library:UCC28180D
- removed J1, J2, J4: Conn_01x02_Pin, Connector_Molex:Molex_KK-254_AE-6410-02A_1x02_P2.54mm_Vertical, symbol Connector:Conn_01x02_Pin
- removed J3: Conn_01x04_Pin, Connector_Molex:Molex_KK-254_AE-6410-04A_1x04_P2.54mm_Vertical, symbol Connector:Conn_01x04_Pin
- removed Q1: IMBG120R234M2HXTMA1, Package_TO_SOT_SMD:TO-263-7_TabPin8, symbol Transistor_FET:C2M1000170J
- removed Q2, Q3: T2N7002AK, Package_TO_SOT_SMD:SOT-23, symbol Transistor_FET:T2N7002AK
- removed Q5, Q6, Q7, Q8: (no value), Package_TO_SOT_THT:TO-247-4_Horizontal_TabDown, symbol Transistor_FET:C3M0030090K
- removed R1: R, symbol Device:R
- removed R10, R11, R12: 5.1k 0.1%, Resistor_SMD:R_0805_2012Metric, symbol Device:R
- removed R13: 10k, Resistor_SMD:R_0805_2012Metric, symbol Device:R
- removed R14: 1k, Resistor_SMD:R_0805_2012Metric, symbol Device:R
- removed R2, R3, R4, R5: 200k, Resistor_SMD:R_2512_6332Metric, symbol Device:R
- removed R6, R7, R8, R9: 1R, Resistor_SMD:R_0805_2012Metric, symbol Device:R
- removed RV1: R_Potentiometer_Trim, Potentiometer_THT:Potentiometer_Vishay_T93YA_Vertical, symbol Device:R_Potentiometer_Trim
- removed TH1: 5k b~=3450, Resistor_SMD:R_0805_2012Metric, symbol Device:Thermistor_NTC
- removed U1, U2: MGJ2D241505SC, Converter_DCDC:Converter_DCDC_Murata_MGJ2DxxxxxxSC_THT, symbol Converter_DCDC_Isolated:MGJ2D241505SC
- removed U3: UCC21520DW, Package_SO:SOIC-16W_7.5x10.3mm_P1.27mm, symbol Driver_FET:UCC21520DW
- removed U4: L7805, digikey-footprints:TO-252-3, symbol Regulator_Linear:L7805
- removed U5: MCP6002-xSN, Package_SO:SOIC-8_3.9x4.9mm_P1.27mm, symbol Amplifier_Operational:MCP6002-xSN
- removed U6: MCP6567, symbol Comparator:MCP6567
- removed U7: 74AHC1G14, Package_TO_SOT_SMD:SOT-23-5, symbol 74xGxx:74AHC1G14
- removed U8: EL817, Package_DIP:DIP-4_W7.62mm, symbol Isolator:EL817
Other:
- added sheet Bridge (bridge.kicad_sch)
- added sheet OTP (otp.kicad_sch)
- added sheet PWM (pwm.kicad_sch)
- added sheet Power (power.kicad_sch)
- added sheet Sense (sense.kicad_sch)

Commit message: voltage sense
Other:
- sheet OTP ports: added CHARGING; removed none
- sheet Sense ports: added CHARGING, VSENSE; removed none
Changed lines of the file:
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@@
 	(generator_version "10.0")
 	(paper "A5")
-	(wire
-		(pts
-			(xy 99.06 74.93) (xy 114.3 74.93)
+	(junction
+		(at 107.95 69.85)
+		(diameter 0)
+		(color 0 0 0 0)
+	)
+	(wire
+		(pts
+			(xy 99.06 95.25) (xy 114.3 95.25)
+		)
+		(stroke
+			(width 0)
+			(type default)
+		)
+	)
+	(wire
+		(pts
+			(xy 107.95 92.71) (xy 107.95 69.85)
+		)
+		(stroke
+			(width 0)
+			(type default)
+		)
+	)
+	(wire
+		(pts
+			(xy 99.06 69.85) (xy 107.95 69.85)
 		)
 		(stroke
@@
 	(wire
 		(pts
+			(xy 99.06 92.71) (xy 107.95 92.71)
+		)
+		(stroke
+			(width 0)
+			(type default)
+		)
+	)
+	(wire
+		(pts
+			(xy 99.06 67.31) (xy 114.3 67.31)
+		)
+		(stroke
+			(width 0)
+			(type default)
+		)
+	)
+	(wire
+		(pts
 			(xy 111.76 63.5) (xy 111.76 48.26)
 		)
@@
 	(wire
 		(pts
+			(xy 107.95 69.85) (xy 114.3 69.85)
+		)
+		(stroke
+			(width 0)
+			(type default)
+		)
+	)
+	(wire
+		(pts
 			(xy 109.22 60.96) (xy 99.06 60.96)
 		)
@@
 	)
 	(sheet
-		(at 86.36 71.12)
-		(size 12.7 7.62)
+		(at 86.36 88.9)
+		(size 12.7 10.16)
 		(exclude_from_sim no)
 		(in_bom yes)
@@
 		)
 		(property "Sheetname" "OTP"
-			(at 86.36 70.4084 0)
+			(at 86.36 88.1884 0)
 			(show_name no)
 			(do_not_autoplace no)
@@
 		)
 		(property "Sheetfile" "otp.kicad_sch"
-			(at 86.36 79.3246 0)
+			(at 86.36 99.6446 0)
 			(show_name no)
 			(do_not_autoplace no)
@@
 		)
 		(pin "~{EN}" input
-			(at 99.06 74.93 0)
+			(at 99.06 95.25 0)
+			(effects
+				(font
+					(size 1.27 1.27)
+				)
+				(justify right)
+			)
+		)
+		(pin "CHARGING" input
+			(at 99.06 92.71 0)
 			(effects
 				(font
@@
 	(sheet
 		(at 86.36 58.42)
-		(size 12.7 7.62)
+		(size 12.7 16.51)
 		(exclude_from_sim no)
 		(in_bom yes)
@@
 		)
 		(property "Sheetfile" "sense.kicad_sch"
-			(at 86.36 66.6246 0)
+			(at 86.36 75.5146 0)
 			(show_name no)
 			(do_not_autoplace no)
@@
 		(pin "CT-" input
 			(at 99.06 63.5 0)
+			(effects
+				(font
+					(size 1.27 1.27)
+				)
+				(justify right)
+			)
+		)
+		(pin "VSENSE" input
+			(at 99.06 67.31 0)
+			(effects
+				(font
+					(size 1.27 1.27)
+				)
+				(justify right)
+			)
+		)
+		(pin "CHARGING" input
+			(at 99.06 69.85 0)
 			(effects
 				(font
@@
 	(sheet
 		(at 114.3 40.64)
-		(size 20.32 38.1)
+		(size 20.32 58.42)
 		(exclude_from_sim no)
 		(in_bom yes)
@@
 		)
 		(property "Sheetfile" "pwm.kicad_sch"
-			(at 114.3 79.3246 0)
+			(at 114.3 99.6446 0)
 			(show_name no)
 			(do_not_autoplace no)
@@
 		)
 		(pin "VSENSE" input
-			(at 114.3 63.5 180)
+			(at 114.3 67.31 180)
 			(effects
 				(font
@@
 		)
 		(pin "CHARGING" input
-			(at 114.3 60.96 180)
+			(at 114.3 69.85 180)
 			(effects
 				(font
@@
 		)
 		(pin "ISENSE" input
-			(at 114.3 66.04 180)
+			(at 114.3 72.39 180)
 			(effects
 				(font
@@
 		)
 		(pin "~{EN}" input
-			(at 114.3 74.93 180)
-			(effects
-				(font
+			(at 114.3 95.25 180)
+			(effects
+				(font

Commit message: finish initial schematic
Other:
- sheet Bridge ports: added I_REF, I_SENSE; removed CT+, CT-
- sheet PWM ports: added ISENSE_CHG, ISENSE_PFC; removed ISENSE
- sheet Sense ports: added ISENSE_CHG, ISENSE_PFC, I_REF, I_SENSE; removed CT+, CT-
Changed lines of the file:
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@@
+	(wire
+		(pts
+			(xy 99.06 74.93) (xy 114.3 74.93)
+		)
+		(stroke
+			(width 0)
+			(type default)
+		)
+	)
 	(wire
 		(pts
@@
 	(wire
 		(pts
+			(xy 99.06 72.39) (xy 114.3 72.39)
+		)
+		(stroke
+			(width 0)
+			(type default)
+		)
+	)
+	(wire
+		(pts
 			(xy 111.76 48.26) (xy 99.06 48.26)
 		)
@@
 	)
 	(sheet
-		(at 86.36 88.9)
-		(size 12.7 10.16)
+		(at 85.09 88.9)
+		(size 13.97 10.16)
 		(exclude_from_sim no)
 		(in_bom yes)
@@
 		)
 		(property "Sheetname" "OTP"
-			(at 86.36 88.1884 0)
+			(at 85.09 88.1884 0)
 			(show_name no)
 			(do_not_autoplace no)
@@
 		)
 		(property "Sheetfile" "otp.kicad_sch"
-			(at 86.36 99.6446 0)
+			(at 85.09 99.6446 0)
 			(show_name no)
 			(do_not_autoplace no)
@@
 	)
 	(sheet
-		(at 86.36 58.42)
-		(size 12.7 16.51)
+		(at 85.09 58.42)
+		(size 13.97 19.05)
 		(exclude_from_sim no)
 		(in_bom yes)
@@
 		)
 		(property "Sheetname" "Sense"
-			(at 86.36 57.7084 0)
+			(at 85.09 57.7084 0)
 			(show_name no)
 			(do_not_autoplace no)
@@
 		)
 		(property "Sheetfile" "sense.kicad_sch"
-			(at 86.36 75.5146 0)
+			(at 85.09 78.0546 0)
 			(show_name no)
 			(do_not_autoplace no)
@@
 				)
 				(justify left top)
-			)
-		)
-		(pin "CT+" input
-			(at 99.06 60.96 0)
-			(effects
-				(font
-					(size 1.27 1.27)
-				)
-				(justify right)
-			)
-		)
-		(pin "CT-" input
-			(at 99.06 63.5 0)
-			(effects
-				(font
-					(size 1.27 1.27)
-				)
-				(justify right)
 			)
 		)
@@
 		(pin "CHARGING" input
 			(at 99.06 69.85 0)
+			(effects
+				(font
+					(size 1.27 1.27)
+				)
+				(justify right)
+			)
+		)
+		(pin "I_REF" input
+			(at 99.06 63.5 0)
+			(effects
+				(font
+					(size 1.27 1.27)
+				)
+				(justify right)
+			)
+		)
+		(pin "I_SENSE" input
+			(at 99.06 60.96 0)
+			(effects
+				(font
+					(size 1.27 1.27)
+				)
+				(justify right)
+			)
+		)
+		(pin "ISENSE_CHG" input
+			(at 99.06 74.93 0)
+			(effects
+				(font
+					(size 1.27 1.27)
+				)
+				(justify right)
+			)
+		)
+		(pin "ISENSE_PFC" input
+			(at 99.06 72.39 0)
 			(effects
 				(font
@@
 	)
 	(sheet
-		(at 86.36 40.64)
-		(size 12.7 12.7)
+		(at 85.09 40.64)
+		(size 13.97 12.7)
 		(exclude_from_sim no)
 		(in_bom yes)
@@
 		)
 		(property "Sheetname" "Bridge"
-			(at 86.36 39.9284 0)
+			(at 85.09 39.9284 0)
 			(show_name no)
 			(do_not_autoplace no)
@@
 		)
 		(property "Sheetfile" "bridge.kicad_sch"
-			(at 86.36 53.9246 0)
+			(at 85.09 53.9246 0)
 			(show_name no)
 			(do_not_autoplace no)
@@
 			)
 		)
-		(pin "CT-" input
+		(pin "I_REF" input
 			(at 99.06 48.26 0)
 			(effects
@@
 			)
 		)
-		(pin "CT+" input
+		(pin "I_SENSE" input
 			(at 99.06 50.8 0)
 			(effects
@@
 			)
 		)
-		(pin "ISENSE" input
-			(at 114.3 72.39 180)
-			(effects
-				(font
-					(size 1.27 1.27)
-				)
-				(justify left)
-			)
-		)
 		(pin "~{EN}" input
 			(at 114.3 95.25 180)
 			(effects
 				(font
+					(size 1.27 1.27)
+				)
+				(justify left)
+			)
+		)
+		(pin "ISENSE_CHG" input
+			(at 114.3 74.93 180)
+			(effects
+				(font
+					(size 1.27 1.27)
+				)
+				(justify left)
+			)
+		)
+		(pin "ISENSE_PFC" input
+			(at 114.3 72.39 180)
+			(effects
+				(font

Commit message: pcb work
Parts:
- added H1, H2, H3, H4: MountingHole_Pad, MountingHole:MountingHole_4.3mm_M4_Pad_Via, symbol Mechanical:MountingHole_Pad
Connections:
- no-connect marks 0 -> 4
