File: PFC.kicad_pcb (KiCad board)
At the start: 2 copper layers, 103 parts, among them IC1 UCC28180D, J1 Conn_01x02_Pin, J10 74650094, J2 Conn_01x02_Pin, J3 Conn_01x04_Pin, J4 Conn_01x02_Pin, J5 74650094, J6 74650094, J7 74650094, J8 74650094, J9 74650094, Q1 IMBG120R234M2HXTMA1, Q2 T2N7002AK, Q3 T2N7002AK, Q4 T2N7002AK, U1 MGJ2D241505SC, U10 MCP6561T-E/OT, U11 MGJ2D241505SC, U12 MCP6562, U13 HOB_50-P, U14 OPA2156ID, U15 OPA2156ID, U16 MCP6562, U17 74LVC1G02, U18 74LVC1G02, U2 MGJ2D241505SC, U3 UCC21520DW, U4 L7805, U5 MCP6002-xSN, U6 74AHC1G32, U7 74AHC1G32, U8 EL817, U9 CD4053B

Commit message: pcb work
Parts:
- removed C14: 1n, Capacitor_SMD:C_0805_2012Metric
- removed J2: Conn_01x02_Pin, Connector_Molex:Molex_KK-254_AE-6410-02A_1x02_P2.54mm_Vertical
- removed RV1: R_Potentiometer_Trim, Potentiometer_THT:Potentiometer_Vishay_T93YA_Vertical
- removed U8: EL817, Package_DIP:DIP-4_W7.62mm
- added C19: 0.1u, Capacitor_SMD:C_0805_2012Metric, B.Cu at (223.8, 127.5)
- added C20: 0.1u, Capacitor_SMD:C_0805_2012Metric, B.Cu at (213.9, 132.0)
- added C21: 0.1u, Capacitor_SMD:C_0805_2012Metric, B.Cu at (94.4, 221.6)
- added C22: 0.1u, Capacitor_SMD:C_0805_2012Metric, B.Cu at (94.4, 224.6)
- added C23: 0.1u, Capacitor_SMD:C_0805_2012Metric, B.Cu at (209.5, 117.5)
- added C24: 0.1u, Capacitor_SMD:C_0805_2012Metric, B.Cu at (227.6, 146.5)
- added C25: 0.1u, Capacitor_SMD:C_0805_2012Metric, B.Cu at (100.9, 219.6)
- added C26: 0.1u, Capacitor_SMD:C_0805_2012Metric, B.Cu at (187.9, 116.2)
- added C27: 0.1u, Capacitor_SMD:C_0805_2012Metric, B.Cu at (175.9, 116.2)
- added C28: 0.1u, Capacitor_SMD:C_0805_2012Metric, B.Cu at (191.5, 122.5)
- added C29: MKS4O141006G00KSSD, Capacitor_THT:C_Rect_L31.5mm_W17.0mm_P27.50mm_MKS4, F.Cu at (237.2, 98.7)
- added D8: LED_Yellow, LED_SMD:LED_0805_2012Metric, B.Cu at (116.7, 169.0)
- added D9: LED_Red, LED_SMD:LED_0805_2012Metric, B.Cu at (116.7, 172.1)
- added H1: MountingHole_Pad, MountingHole:MountingHole_4.3mm_M4_Pad_Via, F.Cu at (109.0, 130.0)
- added H2: MountingHole_Pad, MountingHole:MountingHole_4.3mm_M4_Pad_Via, F.Cu at (109.0, 59.0)
- added H3: MountingHole_Pad, MountingHole:MountingHole_4.3mm_M4_Pad_Via, F.Cu at (250.0, 130.0)
- added H4: MountingHole_Pad, MountingHole:MountingHole_4.3mm_M4_Pad_Via, F.Cu at (250.0, 59.0)
- added R1: 1k, Resistor_SMD:R_0805_2012Metric, B.Cu at (112.3, 169.0)
- added R43: 5.1k 0.1%, Resistor_SMD:R_0805_2012Metric, B.Cu at (188.0, 120.5)
- added R44: 2k 0.1%, Resistor_SMD:R_0805_2012Metric, B.Cu at (191.5, 120.5)
- added R45: 1k, Resistor_SMD:R_0805_2012Metric, B.Cu at (112.3, 171.9)
- added R46: 100R, Resistor_SMD:R_0805_2012Metric, B.Cu at (116.8, 177.1)
- added RV4: 5k, Library:Potentiometer_Bourns_3314G_Vertical_800_400, F.Cu at (112.5, 102.0)
- added RV5: 5k, Library:Potentiometer_Bourns_3314G_Vertical_100_10, F.Cu at (112.5, 118.0)
- added U19: TCMT1100, Package_SO:SOP-4_4.4x2.6mm_P1.27mm, B.Cu at (174.0, 121.5)
- C10, C11, C12, C13, C15, C3, C4, C5, C6, C7, C8, C9, D3, D4, D5, D6, D7, IC1, Q1, Q2, Q3, Q4, R10, R11, R12, R13, R14, R15, R16, R17, R18, R19, R2, R20, R21, R22, R23, R24, R25, R26, R27, R28, R29, R3, R30, R31, R32, R33, R34, R35, R36, R37, R38, R39, R4, R40, R41, R42, R5, R6, R7, R8, R9, TH1, U10, U12, U14, U15, U16, U17, U18, U3, U5, U6, U7, U9: moved to B.Cu
- C16: value 1n -> 0.1u; moved to B.Cu
- C17: value MKP1848C65090JY -> MKP1848C62090JP4; footprint Library:MKP1848C64590JY5_VIS -> Library:MKP1848C62090JP4
- J1: value Conn_01x02_Pin -> Screw_Terminal_01x01; footprint Connector_Molex:Molex_KK-254_AE-6410-02A_1x02_P2.54mm_Vertical -> TerminalBlock_Wuerth:Wuerth_REDCUBE-THR_WP-THRBU_74650074_THR
- U4: footprint digikey-footprints:TO-252-3 -> Package_TO_SOT_SMD:TO-252-2; moved to B.Cu
- moved J1 292.2 mm to (246.6, 92.1)
- moved R5 252.4 mm to (235.5, 102.5), turned to 180 degrees
- moved R4 243.8 mm to (227.5, 102.5), turned to 180 degrees
- moved Q2 242.3 mm to (210.0, 92.4), turned to 90 degrees
- moved D3 241.6 mm to (210.0, 96.0), turned to 180 degrees
- moved Q1 237.7 mm to (223.6, 93.2)
- moved R3 235.3 mm to (219.5, 102.5), turned to 180 degrees
- moved R19 230.8 mm to (235.5, 107.0), turned to 180 degrees
- moved R2 226.9 mm to (211.5, 102.5), turned to 180 degrees
- moved R20 223.2 mm to (227.5, 107.0), turned to 180 degrees
- moved R30 219.9 mm to (229.8, 120.0), turned to 90 degrees
- moved R13 216.6 mm to (227.8, 120.0), turned to -90 degrees
- moved R33 215.8 mm to (231.8, 131.0), turned to 90 degrees
- moved R21 215.8 mm to (219.5, 107.0), turned to 180 degrees
- moved R34 214.0 mm to (229.8, 131.0), turned to -90 degrees
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Connections:
- C16 pad 1: Net-(U15B--) -> Net-(U12B-+)
- C18 pad 1: /Bridge/VIN -> VIN
- J1 pad 1: VBUS -> Net-(J1-Pin_1)
- J7 pad 1: /Bridge/VIN -> VIN
- Q1 pad 8: Net-(J2-Pin_1) -> Net-(J1-Pin_1)
- Q5 pad 1: /Bridge/VIN -> VIN
- Q6 pad 1: /Bridge/VIN -> VIN
- R32 pad 1: /PWM/ISENSE_CHG -> Net-(R32-Pad1)
- R39 pad 2: Net-(U15B--) -> GND
- U14 pad 1: /PWM/ISENSE_CHG -> Net-(R32-Pad1)
- U15 pad 6: Net-(U15B--) -> GND
- U15 pad 7: Net-(U15B--) -> GND
- U3 pad 10: /Bridge/PFC_GATE -> /Bridge/CHSW_GATE
- U3 pad 11: PFC+ -> CHSW+
- U3 pad 14: CHSW- -> PFC-
- U3 pad 15: /Bridge/CHSW_GATE -> /Bridge/PFC_GATE
- U3 pad 16: CHSW+ -> PFC+
- U3 pad 9: PFC- -> CHSW-
- U9 pad 14: Net-(U3-INB) -> Net-(U3-INA)
- U9 pad 15: Net-(U3-INA) -> Net-(U3-INB)
Routing:
- net Net-(J1-Pin_1): track 0.00 -> 42.8 mm
- net GND: track 0.00 -> 34.4 mm, vias 0 -> 11
- net Net-(U12A-+): track 0.00 -> 17.7 mm
- net Net-(D3-K): track 0.00 -> 17.1 mm
- net /PWM/ISENSE_CHG: track 0.00 -> 16.0 mm
- net Net-(Q3-D): track 0.00 -> 15.8 mm
- net Net-(U12A--): track 0.00 -> 14.2 mm
- net /PWM/SET: track 0.00 -> 13.6 mm
- net VBUS: track 0.00 -> 13.3 mm
- net +5V: track 0.00 -> 12.9 mm
- net Net-(U12-Pad1): track 0.00 -> 11.7 mm, vias 0 -> 2
- net -5V: track 0.00 -> 11.0 mm
- net /Bridge/I_REF: track 0.00 -> 9.92 mm
- net Net-(U12B-+): track 0.00 -> 9.57 mm
- net /Sense/I_REF_BUF: track 0.00 -> 9.43 mm
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- added copper zone on F.Cu, net /Bridge/L1
- added copper zone on F.Cu, net /Bridge/L2_CS
- added copper zone on F.Cu, net GND
- added copper zone on In1.Cu, net GND
- added copper zone on F.Cu, net VBUS
- added copper zone on B.Cu, net VIN
Other:
- board outline added: 150 x 80 mm
- copper layers 2 -> 4
- board text added: "Irms (A)"
- board text added: "Vbus (V)"

Commit message: logic layout
Parts:
- added C30: 0.1u, Capacitor_SMD:C_0805_2012Metric, B.Cu at (182.0, 103.5)
- moved Q4 169.2 mm to (225.0, 117.5)
- moved C3 162.7 mm to (224.5, 120.5)
- moved C4 153.1 mm to (213.5, 123.0), turned to 0 degrees
- moved C5 152.4 mm to (210.0, 121.0), turned to 0 degrees
- moved C25 148.4 mm to (210.1, 119.0), turned to 0 degrees
- moved U9 146.0 mm to (205.0, 113.0), turned to 90 degrees
- moved R17 140.0 mm to (224.5, 122.5), turned to 0 degrees
- moved R15 136.8 mm to (221.1, 117.0)
- moved R16 134.9 mm to (217.5, 117.0), turned to 0 degrees
- moved C15 132.9 mm to (224.5, 126.5), turned to 0 degrees
- moved R18 132.4 mm to (213.5, 121.0)
- moved C6 125.6 mm to (224.5, 124.5)
- moved U10 121.9 mm to (195.4, 125.0)
- moved R38 120.3 mm to (198.5, 129.5), turned to 90 degrees
- moved D7 118.8 mm to (175.0, 117.5), turned to 0 degrees
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Connections:
- R39 pad 2: GND -> Net-(U15B--)
- R46 pad 1: unconnected-(R46-Pad1) -> /PWM/ISENSE_CHG
- R46 pad 2: unconnected-(R46-Pad2) -> Net-(R32-Pad1)
- U15 pad 6: GND -> Net-(U15B--)
- U15 pad 7: GND -> Net-(U15B--)
Routing:
- net /PWM/VSENSE: track 0.00 -> 153.7 mm, vias 0 -> 3
- net Net-(R22-Pad2): track 0.00 -> 145.1 mm, vias 0 -> 3
- net Net-(U10--): track 0.00 -> 123.2 mm, vias 0 -> 2
- net Net-(R37-Pad1): track 0.00 -> 112.4 mm, vias 0 -> 1
- net Net-(R38-Pad2): track 0.00 -> 98.5 mm, vias 0 -> 1
- net Net-(U10-+): track 0.00 -> 92.0 mm
- net Net-(U15B-+): track 0.00 -> 88.1 mm, vias 0 -> 1
- net GND: track 34.4 -> 118.4 mm, vias 11 -> 22
- net /PWM/ISENSE_PFC: track 0.00 -> 75.2 mm, vias 0 -> 4
- net Net-(U3-INA): track 0.00 -> 61.7 mm
- net /Sense/I_REF_BUF: track 9.43 -> 57.8 mm, vias 0 -> 3
- net +5V: track 12.9 -> 59.5 mm, vias 0 -> 11
- net /OTP/CHARGING: track 0.00 -> 44.1 mm, vias 0 -> 2
- net Net-(U3-INB): track 0.00 -> 43.3 mm
- net /Bridge/I_SENSE: track 4.78 -> 47.5 mm, vias 0 -> 2
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- added copper zone on In2.Cu, net +5V
- added copper zone on F.Cu, net /Bridge/L2
- added copper zone on B.Cu, net GND

Commit message: layout work
Parts:
- removed U12: MCP6562, Package_SO:SOIC-8_3.9x4.9mm_P1.27mm
- removed U5: MCP6002-xSN, Package_SO:SOIC-8_3.9x4.9mm_P1.27mm
- added C1: 10u, Capacitor_SMD:C_1210_3225Metric, B.Cu at (134.0, 118.0)
- added C14: 10u, Capacitor_SMD:C_1210_3225Metric, B.Cu at (129.0, 118.0)
- added C2: 10u, Capacitor_SMD:C_1210_3225Metric, B.Cu at (174.5, 94.5)
- added C31: 10u, Capacitor_SMD:C_1210_3225Metric, B.Cu at (190.5, 94.5)
- added C32: 10u, Capacitor_SMD:C_1210_3225Metric, B.Cu at (190.5, 91.0)
- added C33: 10u, Capacitor_SMD:C_1210_3225Metric, B.Cu at (129.0, 128.5)
- added C34: 10u, Capacitor_SMD:C_1210_3225Metric, B.Cu at (133.5, 107.5)
- added C35: 10u, Capacitor_SMD:C_1210_3225Metric, B.Cu at (128.5, 111.0)
- added C36: 10u, Capacitor_SMD:C_1210_3225Metric, B.Cu at (133.5, 111.0)
- added C37: 10u, Capacitor_SMD:C_1210_3225Metric, B.Cu at (128.5, 107.5)
- added C38: 10u, Capacitor_SMD:C_1210_3225Metric, B.Cu at (90.0, 132.4)
- added C39: 10u, Capacitor_SMD:C_1210_3225Metric, B.Cu at (90.0, 136.6)
- added C40: 10u, Capacitor_SMD:C_1210_3225Metric, B.Cu at (120.0, 118.0)
- added C41: 10u, Capacitor_SMD:C_1210_3225Metric, B.Cu at (120.0, 111.0)
- added C42: 10u, Capacitor_SMD:C_1210_3225Metric, B.Cu at (120.0, 107.5)
- added C43: 10u, Capacitor_SMD:C_1210_3225Metric, B.Cu at (120.0, 132.0)
- added C44: 10u, Capacitor_SMD:C_1210_3225Metric, B.Cu at (120.0, 128.5)
- added C45: 10u, Capacitor_SMD:C_1210_3225Metric, B.Cu at (120.0, 121.5)
- added C46: 10u, Capacitor_SMD:C_1210_3225Metric, B.Cu at (134.0, 132.0)
- added C47: 10u, Capacitor_SMD:C_1210_3225Metric, B.Cu at (129.0, 132.0)
- added C48: 10u, Capacitor_SMD:C_1210_3225Metric, B.Cu at (134.0, 121.5)
- added C49: 10u, Capacitor_SMD:C_1210_3225Metric, B.Cu at (129.0, 121.5)
- added D10: BAT42W-V, Diode_SMD:D_SOD-123, B.Cu at (74.6, 89.0)
- added D11: BAT42W-V, Diode_SMD:D_SOD-123, B.Cu at (74.6, 92.4)
- added D12: BAT42W-V, Diode_SMD:D_SOD-123, B.Cu at (74.6, 95.7)
- added D13: BAT42W-V, Diode_SMD:D_SOD-123, B.Cu at (186.5, 131.5)
- added J11: Conn_01x02_Pin, Connector_Molex:Molex_KK-254_AE-6410-02A_1x02_P2.54mm_Vertical, F.Cu at (158.5, 130.8)
- added R47: 1M, Resistor_SMD:R_0805_2012Metric, B.Cu at (69.5, 85.5)
- added R48: 1M, Resistor_SMD:R_0805_2012Metric, B.Cu at (69.5, 88.4)
- added R49: 1M, Resistor_SMD:R_0805_2012Metric, B.Cu at (194.5, 120.0)
- added U8: MCP6001-OT, Package_TO_SOT_SMD:SOT-23-5, B.Cu at (182.0, 131.0)
- C21, C22: value 0.1u -> 10u; footprint Capacitor_SMD:C_0805_2012Metric -> Capacitor_SMD:C_1210_3225Metric
- C7: value 1n -> 0.1u
- D4: value BAT54C -> BAT42W-V; footprint Package_TO_SOT_SMD:SOT-23 -> Diode_SMD:D_SOD-123
- U6: value 74AHC1G32 -> MCP6561-OT
- moved R45 119.5 mm to (225.0, 132.0), turned to 90 degrees
- moved R1 119.2 mm to (224.5, 128.5)
- moved D8 118.2 mm to (229.0, 132.0), turned to 90 degrees
- moved D9 117.3 mm to (227.0, 132.0), turned to 90 degrees
- moved R9 116.7 mm to (193.5, 85.0), turned to 0 degrees
- moved C21 111.4 mm to (174.5, 91.0), turned to 0 degrees
- moved R8 105.1 mm to (177.0, 82.4), turned to 90 degrees
- moved C22 76.3 mm to (134.0, 128.5)
- moved U19 35.4 mm to (152.5, 118.0), turned to -90 degrees
- moved U6 33.7 mm to (69.1, 92.3), turned to 180 degrees
- moved D4 25.2 mm to (74.6, 85.7), turned to 180 degrees
- moved Q3 24.0 mm to (66.9, 107.7)
- moved C10 21.5 mm to (60.2, 107.0)
- moved C11 20.6 mm to (60.2, 110.0), turned to 180 degrees
- moved R14 15.2 mm to (76.0, 115.8), turned to 180 degrees
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Connections:
- C21 pad 1: +5V -> CHSW_GND
- C21 pad 2: GND -> CHSW-
- C22 pad 1: +5V -> PFC+
- C22 pad 2: GND -> PFC_GND
- C26 pad 1: Net-(J3-Pin_2) -> Net-(D4-A)
- C7 pad 2: Net-(U10-+) -> Net-(D13-K)
- D4 pad 1: Net-(D4-Pad1) -> Net-(D10-K)
- D4 pad 2: Net-(D4-Pad2) -> Net-(D4-A)
- J3 pad 2: Net-(J3-Pin_2) -> Net-(D4-A)
- R10 pad 1: Net-(J3-Pin_2) -> Net-(D4-A)
- R28 pad 1: Net-(U10-+) -> Net-(U8-+)
- R29 pad 2: Net-(U10-+) -> Net-(U8-+)
- U1 pad 1: unconnected-(U1-+VIN-Pad1) -> 24V_IN
- U1 pad 2: unconnected-(U1--VIN-Pad2) -> GND_IN
- U10 pad 3: Net-(U10-+) -> Net-(D13-K)
- U11 pad 1: unconnected-(U11-+VIN-Pad1) -> 24V_IN
- U11 pad 2: unconnected-(U11--VIN-Pad2) -> GND_IN
- U19 pad 3: Net-(J4-Pin_1) -> Net-(J4-Pin_2)
- U19 pad 4: Net-(J4-Pin_2) -> Net-(J4-Pin_1)
- U2 pad 1: unconnected-(U2-+VIN-Pad1) -> 24V_IN
- U2 pad 2: unconnected-(U2--VIN-Pad2) -> GND_IN
- U6 pad 1: Net-(U12-Pad1) -> /OTP/~{EN}
- U6 pad 2: Net-(U12-Pad7) -> GND
- U6 pad 3: GND -> Net-(D10-K)
- U6 pad 4: /OTP/~{EN} -> Net-(D12-K)
Routing:
- net PFC_GND: track 0.00 -> 142.6 mm, vias 0 -> 1
- net CHSW_GND: track 0.00 -> 121.7 mm, vias 0 -> 1
- net Net-(U10-+): track 92.0 -> 0.00 mm
- net PFC+: track 0.00 -> 89.0 mm, vias 0 -> 1
- net PFC-: track 0.00 -> 83.6 mm, vias 0 -> 1
- net CHSW-: track 0.00 -> 73.3 mm, vias 0 -> 1
- net 24V_IN: track 0.00 -> 72.7 mm
- net Net-(U8-+): track 0.00 -> 70.1 mm
- net GND_IN: track 0.00 -> 69.2 mm
- net CHSW+: track 0.00 -> 68.3 mm, vias 0 -> 1
- net /Bridge/CHSW_GATE: track 0.00 -> 55.2 mm, vias 0 -> 2
- net /Bridge/L1: track 0.00 -> 55.0 mm, vias 0 -> 6
- net +5V: track 59.5 -> 88.4 mm, vias 11 -> 12
- net /Bridge/PFC_GATE: track 0.00 -> 28.2 mm, vias 0 -> 2
- net Net-(D13-K): track 0.00 -> 24.4 mm
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
Commit message: otp layout
Parts:
- removed D12: BAT42W-V, Diode_SMD:D_SOD-123
- removed R48: 1M, Resistor_SMD:R_0805_2012Metric
- added C50: 10u, Capacitor_SMD:C_1210_3225Metric, B.Cu at (190.0, 126.0)
- added C51: 0.1u, Capacitor_SMD:C_0805_2012Metric, B.Cu at (145.2, 120.0)
- added C52: 0.1u, Capacitor_SMD:C_0805_2012Metric, B.Cu at (139.0, 124.0)
- moved C28 124.9 mm to (196.5, 117.5), turned to 0 degrees
- moved C11 119.6 mm to (178.5, 128.0)
- moved U7 118.3 mm to (189.5, 122.5)
- moved C10 116.7 mm to (175.0, 128.0)
- moved R47 91.0 mm to (148.5, 130.6), turned to -90 degrees
- moved D4 89.7 mm to (152.0, 131.0), turned to 0 degrees
- moved D10 86.7 mm to (152.0, 128.0), turned to 0 degrees
- moved Q3 83.2 mm to (149.0, 121.5), turned to 0 degrees
- moved U6 80.5 mm to (141.5, 127.5)
- moved C27 78.3 mm to (149.0, 125.0), turned to 90 degrees
- moved R11 76.5 mm to (151.0, 125.0), turned to 90 degrees
- moved C26 74.9 mm to (145.0, 125.0), turned to 90 degrees
- moved R10 73.2 mm to (147.0, 125.0), turned to 90 degrees
- moved R14 73.0 mm to (149.0, 118.5), turned to 0 degrees
- moved D11 71.7 mm to (140.5, 120.5)
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Connections:
- C28 pad 1: Net-(D12-A) -> GND
- C28 pad 2: GND -> -5V
- R43 pad 1: Net-(D12-A) -> Net-(U6--)
- R44 pad 2: Net-(D12-A) -> Net-(U6--)
- U6 pad 4: Net-(D12-K) -> Net-(U6--)
Routing:
- net /OTP/~{EN}: track 16.9 -> 158.5 mm, vias 0 -> 4
- net +5V: track 88.4 -> 201.3 mm, vias 12 -> 18
- net -5V: track 18.9 -> 126.3 mm, vias 0 -> 3
- net +15V: track 9.69 -> 117.0 mm, vias 0 -> 2
- net Net-(D11-A): track 0.00 -> 59.3 mm, vias 0 -> 2
- net Net-(Q3-G): track 0.00 -> 57.3 mm, vias 0 -> 2
- net GND: track 140.0 -> 180.3 mm, vias 24 -> 35
- net Net-(D4-A): track 0.00 -> 26.8 mm
- net Net-(D10-A): track 0.00 -> 20.7 mm
- net Net-(D10-K): track 0.00 -> 20.3 mm
- net /OTP/CHARGING: track 57.3 -> 67.4 mm
- net Net-(Q3-D): track 0.00 -> 8.01 mm
- net /Bridge/I_REF: track 5.07 -> 11.6 mm
- net Net-(R14-Pad2): track 0.00 -> 4.50 mm
- net /Bridge/I_SENSE: track 44.9 -> 49.3 mm
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