File: PFC.kicad_pcb (KiCad board)
At the start: 4 copper layers, 150 x 80 mm, 155 parts, among them IC1 UCC28180D, J1 Screw_Terminal_01x01, J10 74650094, J11 Conn_01x02_Pin, J3 Conn_01x04_Pin, J4 Conn_01x02_Pin, J5 74650094, J6 74650094, J7 74650094, J8 74650094, J9 74650094, Q1 IMBG120R234M2HXTMA1, Q2 T2N7002AK, Q3 T2N7002AK, Q4 T2N7002AK, U1 MGJ2D241505SC, U10 MCP6561T-E/OT, U11 MGJ2D241505SC, U13 HOB_50-P, U14 OPA2156ID, U15 OPA2156ID, U16 MCP6562, U17 74LVC1G02, U18 74LVC1G02, U19 TCMT1100, U2 MGJ2D241505SC, U3 UCC21520DW, U4 L7805, U6 MCP6561-OT, U7 74AHC1G32, U8 MCP6001-OT, U9 CD4053B

Commit message: solder mask
Routing:
- net Net-(J1-Pin_1): track 48.0 -> 0.00 mm
- net GND: track 180.3 -> 154.7 mm, vias 35 -> 384
- added copper zone on B.Cu, net /Bridge/L1
- added copper zone on B.Cu, net Net-(J1-Pin_1)
Other:
- outline, holes or cut-outs redrawn

Commit message: final touches?
Parts:
- added TP1: TestPoint, TestPoint:TestPoint_Pad_1.0x1.0mm, B.Cu at (148.5, 128.2)
- added TP2: TestPoint, TestPoint:TestPoint_Pad_1.0x1.0mm, B.Cu at (211.8, 114.5)
- added TP3: TestPoint, TestPoint:TestPoint_Pad_1.0x1.0mm, B.Cu at (214.5, 114.5)
- added TP4: TestPoint, TestPoint:TestPoint_Pad_1.0x1.0mm, B.Cu at (217.2, 114.5)
- added TP5: TestPoint, TestPoint:TestPoint_Pad_1.0x1.0mm, B.Cu at (220.0, 114.5)
- added TP6: TestPoint, TestPoint:TestPoint_Pad_1.0x1.0mm, B.Cu at (225.5, 114.5)
- added TP7: TestPoint, TestPoint:TestPoint_Pad_1.0x1.0mm, B.Cu at (222.8, 114.5)
- moved R47 0.66 mm to (148.5, 131.2)
Routing:
- net /PWM/ISENSE_CHG: track 14.9 -> 47.2 mm, vias 3 -> 4
- net /PWM/ISENSE_PFC: track 75.2 -> 92.2 mm, vias 4 -> 5
- net /PWM/CHG_PWM: track 31.8 -> 35.5 mm
- net GND: track 154.7 -> 157.5 mm, vias 384 -> 367
- net Net-(D10-K): track 20.3 -> 22.9 mm
- net -5V: track 126.3 -> 123.7 mm
- net /PWM/PFC_PWM: track 20.2 -> 22.7 mm, vias 2 -> 3
- net +5V: track 201.3 -> 203.1 mm, vias 18 -> 19
Other:
- outline, holes or cut-outs redrawn
- board text added: "+5V"
- board text added: "CHG"
- board text added: "DSCHG"
- board text added: "GND"
- board text added: "ICHG"
- board text added: "IPFC"
- board text added: "PFC"
- board text added: "Tmax"
- board text added: "VIN"
- board text added: "VOUT"
- board text added: "~{EN}"
