File: bridge.kicad_sch (KiCad schematic)
At the start: 20 parts, among them T1 CST2010, T2 CST2010

Commit message: voltage sense
Connections:
- net GNDPWR is gone; now on net GND: C1.2, C2.2, D5.2 (A), D6.2 (A), Q7.2 (S), Q8.2 (S)
- net GND: no longer Q7.3 (DS), Q8.3 (DS)
- new net PFC_GND: Q7.3 (DS), Q8.3 (DS)
Changed lines of the file:
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@@
+		)
+	)
+	(global_label "PFC_GND"
+		(shape input)
+		(at 138.43 105.41 180)
+		(fields_autoplaced yes)
+		(effects
+			(font
+				(size 1.27 1.27)
+			)
+			(justify right)
+		)
+		(property "Intersheetrefs" "${INTERSHEET_REFS}"
+			(at 126.9781 105.41 0)
+			(hide yes)
+			(show_name no)
+			(do_not_autoplace no)
+			(effects
+				(font
+					(size 1.27 1.27)
+				)
+				(justify right)
+			)
 		)
 	)
@@
 	)
 	(symbol
+		(lib_id "power:GND")
+		(at 90.17 109.22 0)
+		(unit 1)
+		(body_style 1)
+		(exclude_from_sim no)
+		(in_bom yes)
+		(on_board yes)
+		(in_pos_files yes)
+		(dnp no)
+		(fields_autoplaced yes)
+		(property "Reference" "#PWR043"
+			(at 90.17 115.57 0)
+			(hide yes)
+			(show_name no)
+			(do_not_autoplace no)
+			(effects
+				(font
+					(size 1.27 1.27)
+				)
+			)
+		)
+		(property "Value" "GND"
+			(at 90.17 114.3 0)
+			(show_name no)
+			(do_not_autoplace no)
+			(effects
+				(font
+					(size 1.27 1.27)
+				)
+			)
+		)
+		(property "Footprint" ""
+			(at 90.17 109.22 0)
+			(hide yes)
+			(show_name no)
+			(do_not_autoplace no)
+			(effects
+				(font
+					(size 1.27 1.27)
+				)
+			)
+		)
+		(property "Datasheet" ""
+			(at 90.17 109.22 0)
+			(hide yes)
+			(show_name no)
+			(do_not_autoplace no)
+			(effects
+				(font
+					(size 1.27 1.27)
+				)
+			)
+		)
+		(property "Description" "Power symbol creates a global label with name \"GND\" , ground"
+			(at 90.17 109.22 0)
+			(hide yes)
+			(show_name no)
+			(do_not_autoplace no)
+			(effects
+				(font
+					(size 1.27 1.27)
+				)
+			)
+		)
+		(pin "1"
+		)
+		(instances
+			(project "PFC"
+				(path "/9a4457e8-cc73-4b75-ac20-82cc64952613/6eb0d11a-b8cc-4b9f-9b90-475ada58642f"
+					(reference "#PWR043")
+					(unit 1)
+				)
+			)
+		)
+	)
+	(symbol
 		(lib_id "Device:R")
 		(at 93.98 92.71 0)
@@
 					(unit 1)
 				)
-			)
-		)
-	)
-	(symbol
-		(lib_id "power:GND")
-		(at 138.43 105.41 270)
-		(unit 1)
-		(body_style 1)
-		(exclude_from_sim no)
-		(in_bom yes)
-		(on_board yes)
-		(in_pos_files yes)
-		(dnp no)
-		(fields_autoplaced yes)
-		(property "Reference" "#PWR01"
-			(at 132.08 105.41 0)
-			(hide yes)
-			(show_name no)
-			(do_not_autoplace no)
-			(effects
-				(font
-					(size 1.27 1.27)
-				)
-			)
-		)
-		(property "Value" "GND"
-			(at 134.62 105.4099 90)
-			(show_name no)
-			(do_not_autoplace no)
-			(effects
-				(font
-					(size 1.27 1.27)
-				)
-				(justify right)
-			)
-		)
-		(property "Footprint" ""
-			(at 138.43 105.41 0)
-			(hide yes)
-			(show_name no)
-			(do_not_autoplace no)
-			(effects
-				(font
-					(size 1.27 1.27)
-				)
-			)
-		)
-		(property "Datasheet" ""
-			(at 138.43 105.41 0)
-			(hide yes)
-			(show_name no)
-			(do_not_autoplace no)
-			(effects
-				(font
-					(size 1.27 1.27)
-				)
-			)
-		)
-		(property "Description" "Power symbol creates a global label with name \"GND\" , ground"
-			(at 138.43 105.41 0)
-			(hide yes)
-			(show_name no)
-			(do_not_autoplace no)
-			(effects
-				(font
-					(size 1.27 1.27)
-				)
-			)
-		)
-		(pin "1"
-		)
-		(instances
-			(project "PFC"
-				(path "/9a4457e8-cc73-4b75-ac20-82cc64952613/6eb0d11a-b8cc-4b9f-9b90-475ada58642f"
-					(reference "#PWR01")
-					(unit 1)
-				)
-			)
-		)
-	)
-	(symbol
-		(lib_id "power:GNDPWR")
-		(at 90.17 109.22 0)
-		(unit 1)
-		(body_style 1)
-		(exclude_from_sim no)
-		(in_bom yes)
-		(on_board yes)
-		(in_pos_files yes)
-		(dnp no)
-		(fields_autoplaced yes)
-		(property "Reference" "#PWR016"
-			(at 90.17 114.3 0)
-			(hide yes)
-			(show_name no)
-			(do_not_autoplace no)
-			(effects
-				(font
-					(size 1.27 1.27)
-				)
-			)
-		)
-		(property "Value" "GNDPWR"
-			(at 90.043 113.03 0)
-			(show_name no)
-			(do_not_autoplace no)
-			(effects
-				(font
-					(size 1.27 1.27)
-				)
-			)
-		)
-		(property "Footprint" ""
-			(at 90.17 110.49 0)
-			(hide yes)
-			(show_name no)
-			(do_not_autoplace no)
-			(effects
-				(font
-					(size 1.27 1.27)
-				)
-			)
-		)
-		(property "Datasheet" ""
-			(at 90.17 110.49 0)
-			(hide yes)
-			(show_name no)
-			(do_not_autoplace no)
-			(effects
-				(font
-					(size 1.27 1.27)
-				)
-			)
-		)
-		(property "Description" "Power symbol creates a global label with name \"GNDPWR\" , global ground"
-			(at 90.17 109.22 0)
-			(hide yes)
-			(show_name no)
-			(do_not_autoplace no)
-			(effects
-				(font
-					(size 1.27 1.27)
-				)
-			)
-		)
-		(pin "1"
-		)
-		(instances
-			(project "PFC"
-				(path "/9a4457e8-cc73-4b75-ac20-82cc64952613/6eb0d11a-b8cc-4b9f-9b90-475ada58642f"
-					(reference "#PWR016")
-					(unit 1)
-				)

Commit message: finish initial schematic
Parts:
- removed D10, D7, D8, D9: B160-E3, Diode_SMD:D_SMA, symbol Diode:B160-E3
- removed T1, T2: CST2010, Transformer_SMD:Transformer_Coilcraft_CST2010, symbol Transformer:CST2010
- added C9: 0.1u, Capacitor_SMD:C_0805_2012Metric, symbol Device:C
- added J5, J6, J7, J8: 74650094, TerminalBlock_Wuerth:Wuerth_REDCUBE-THR_WP-THRBU_74650094_THR, symbol Connector:Screw_Terminal_01x01
- added U13: HOB_50-P, Library:HOB130P, symbol New_Library:HOB_130-P
Connections:
- net GND: now also C9.2, J8.1 (Pin_1), U13.2 (GND_-_OR_0_V)
- net L1: now also J5.1 (Pin_1)
- net L2: now also J6.1 (Pin_1), U13.6 (IP_IN_1), U13.7 (IP_IN_2), U13.8 (IP_IN_3), U13.9 (IP_IN_4); no longer D1.2 (A), D2.2 (A)
- net VBUS: now also D1.1 (K), D2.1 (K)
- net VIN: now also J7.1 (Pin_1)
- net L2_CS: now reaches Q7.1 (D), Q8.1 (D)
- net L2_CS: now also D1.2 (A), D2.2 (A), U13.10 (IP_OUT_1), U13.11 (IP_OUT_2), U13.12 (IP_OUT_3), U13.13 (IP_OUT_4)
- new net +5V: C9.1, U13.1 (+UC)
- new net I_REF: U13.4 (UREF_(OUT))
- new net I_SENSE: U13.3 (UOUT)
Other:
- moved on the sheet: C2, D1, D2

Commit message: pcb layout
Parts:
- removed C1, C2: C, symbol Device:C
- added C17: MKP1848C65090JY, Library:MKP1848C64590JY5_VIS, symbol Device:C
- added C18: MKS4O141006G00KSSD, Capacitor_THT:C_Rect_L31.5mm_W17.0mm_P27.50mm_MKS4, symbol Device:C
- added J10, J9: 74650094, TerminalBlock_Wuerth:Wuerth_REDCUBE-THR_WP-THRBU_74650094_THR, symbol Connector:Screw_Terminal_01x01
Connections:
- net GND: now also C17.2, C18.2, J10.1 (Pin_1)
- net VBUS: now also C17.1, J9.1 (Pin_1)
- net VIN: now also C18.1

Commit message: pcb work
Parts:
- added C29: MKS4O141006G00KSSD, Capacitor_THT:C_Rect_L31.5mm_W17.0mm_P27.50mm_MKS4, symbol Device:C
- C17: value MKP1848C65090JY -> MKP1848C62090JP4; footprint Library:MKP1848C64590JY5_VIS -> Library:MKP1848C62090JP4
Connections:
- net GND: now also C29.2
- net VBUS: now also C29.1
Changed lines of the file:
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@@
 	(paper "A4")
 	(junction
+		(at 193.04 87.63)
+		(diameter 0)
+		(color 0 0 0 0)
+	)
+	(junction
 		(at 73.66 107.95)
 		(diameter 0)
@@
 	)
 	(junction
+		(at 193.04 100.33)
+		(diameter 0)
+		(color 0 0 0 0)
+	)
+	(junction
 		(at 80.01 80.01)
 		(diameter 0)
@@
 	(wire
 		(pts
+			(xy 193.04 87.63) (xy 201.93 87.63)
+		)
+		(stroke
+			(width 0)
+			(type default)
+		)
+	)
+	(wire
+		(pts
 			(xy 182.88 107.95) (xy 182.88 106.68)
 		)
@@
 	(wire
 		(pts
+			(xy 73.66 77.47) (xy 73.66 80.01)
+		)
+		(stroke
+			(width 0)
+			(type default)
+		)
+	)
+	(wire
+		(pts
 			(xy 113.03 99.06) (xy 113.03 107.95)
 		)
@@
 	(wire
 		(pts
+			(xy 201.93 100.33) (xy 193.04 100.33)
+		)
+		(stroke
+			(width 0)
+			(type default)
+		)
+	)
+	(wire
+		(pts
 			(xy 173.99 104.14) (xy 173.99 105.41)
 		)
@@
 	(wire
 		(pts
+			(xy 201.93 97.79) (xy 201.93 100.33)
+		)
+		(stroke
+			(width 0)
+			(type default)
+		)
+	)
+	(wire
+		(pts
 			(xy 124.46 58.42) (xy 123.19 58.42)
 		)
@@
 	(wire
 		(pts
+			(xy 74.93 77.47) (xy 73.66 77.47)
+		)
+		(stroke
+			(width 0)
+			(type default)
+		)
+	)
+	(wire
+		(pts
 			(xy 109.22 99.06) (xy 109.22 107.95)
 		)
@@
 	(wire
 		(pts
+			(xy 193.04 87.63) (xy 193.04 90.17)
+		)
+		(stroke
+			(width 0)
+			(type default)
+		)
+	)
+	(wire
+		(pts
 			(xy 93.98 97.79) (xy 100.33 97.79)
 		)
@@
 	(wire
 		(pts
-			(xy 193.04 97.79) (xy 193.04 107.95)
+			(xy 193.04 97.79) (xy 193.04 100.33)
 		)
 		(stroke
@@
 	(wire
 		(pts
-			(xy 193.04 80.01) (xy 193.04 90.17)
+			(xy 193.04 80.01) (xy 193.04 87.63)
 		)
 		(stroke
@@
 	(wire
 		(pts
+			(xy 201.93 90.17) (xy 201.93 87.63)
+		)
+		(stroke
+			(width 0)
+			(type default)
+		)
+	)
+	(wire
+		(pts
 			(xy 163.83 97.79) (xy 139.7 97.79)
 		)
@@
 	(wire
 		(pts
+			(xy 193.04 100.33) (xy 193.04 107.95)
+		)
+		(stroke
+			(width 0)
+			(type default)
+		)
+	)
+	(wire
+		(pts
 			(xy 80.01 80.01) (xy 80.01 90.17)
 		)
@@
 			(width 0)
 			(type default)
-		)
-	)
-	(label "VIN"
-		(at 73.66 80.01 0)
-		(effects
-			(font
-				(size 1.27 1.27)
-			)
-			(justify left bottom)
 		)
 	)
@@
 				)
 				(justify right)
+			)
+		)
+	)
+	(global_label "VIN"
+		(shape input)
+		(at 74.93 77.47 0)
+		(fields_autoplaced yes)
+		(effects
+			(font
+				(size 1.27 1.27)
+			)
+			(justify left)
+		)
+		(property "Intersheetrefs" "${INTERSHEET_REFS}"
+			(at 80.9391 77.47 0)
+			(hide yes)
+			(show_name no)
+			(do_not_autoplace no)
+			(effects
+				(font
+					(size 1.27 1.27)
+				)
+				(justify left)
 			)
 		)
@@
 			)
 		)
-		(property "Value" "MKP1848C65090JY"
+		(property "Value" "MKP1848C62090JP4"
 			(at 196.85 95.2499 0)
 			(hide yes)
@@
 			)
 		)
-		(property "Footprint" "Library:MKP1848C64590JY5_VIS"
+		(property "Footprint" "Library:MKP1848C62090JP4"
 			(at 194.0052 97.79 0)
 			(hide yes)
@@
 					(unit 1)
 				)
+			)
+		)
+	)
+	(symbol
+		(lib_id "Device:C")
+		(at 201.93 93.98 0)
+		(unit 1)
+		(body_style 1)
+		(exclude_from_sim no)
+		(in_bom yes)
+		(on_board yes)
+		(in_pos_files yes)
+		(dnp no)
+		(property "Reference" "C29"
+			(at 203.708 91.44 0)
+			(show_name no)
+			(do_not_autoplace no)
+			(effects
+				(font
+					(size 1.27 1.27)
+				)
+				(justify left)
+			)
+		)
+		(property "Value" "MKS4O141006G00KSSD"
+			(at 205.74 95.2499 0)
+			(hide yes)
+			(show_name no)
+			(do_not_autoplace no)
+			(effects
+				(font
+					(size 1.27 1.27)
+				)
+				(justify left)
+			)
+		)
+		(property "Footprint" "Capacitor_THT:C_Rect_L31.5mm_W17.0mm_P27.50mm_MKS4"
+			(at 202.8952 97.79 0)
+			(hide yes)
+			(show_name no)
+			(do_not_autoplace no)
+			(effects
+				(font
+					(size 1.27 1.27)
+				)
+			)
+		)
+		(property "Datasheet" ""
+			(at 201.93 93.98 0)
+			(hide yes)
+			(show_name no)
+			(do_not_autoplace no)
+			(effects
+				(font
+					(size 1.27 1.27)
+				)
+			)
+		)
+		(property "Description" "Unpolarized capacitor"
+			(at 201.93 93.98 0)
+			(hide yes)
+			(show_name no)
+			(do_not_autoplace no)
+			(effects
+				(font
+					(size 1.27 1.27)
+				)
+			)
+		)
+		(pin "2"
+		)
+		(pin "1"
+		)
+		(instances
+			(project "PFC"
+				(path "/9a4457e8-cc73-4b75-ac20-82cc64952613/6eb0d11a-b8cc-4b9f-9b90-475ada58642f"
+					(reference "C29")
+					(unit 1)
+				)

Commit message: final touches?
Changed lines of the file:
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@@
-	)
-	(junction
-		(at 80.01 80.01)
-		(diameter 0)
-		(color 0 0 0 0)
 	)
 	(junction
@@
 	)
 	(junction
-		(at 80.01 107.95)
-		(diameter 0)
-		(color 0 0 0 0)
-	)
-	(junction
 		(at 91.44 80.01)
 		(diameter 0)
@@
 	(wire
 		(pts
-			(xy 80.01 97.79) (xy 80.01 107.95)
-		)
-		(stroke
-			(width 0)
-			(type default)
-		)
-	)
-	(wire
-		(pts
-			(xy 80.01 80.01) (xy 91.44 80.01)
+			(xy 73.66 80.01) (xy 91.44 80.01)
 		)
 		(stroke
@@
 	(wire
 		(pts
-			(xy 73.66 80.01) (xy 80.01 80.01)
-		)
-		(stroke
-			(width 0)
-			(type default)
-		)
-	)
-	(wire
-		(pts
 			(xy 166.37 101.6) (xy 163.83 101.6)
 		)
@@
 	(wire
 		(pts
-			(xy 73.66 107.95) (xy 80.01 107.95)
+			(xy 73.66 107.95) (xy 109.22 107.95)
 		)
 		(stroke
@@
 	(wire
 		(pts
-			(xy 80.01 80.01) (xy 80.01 90.17)
-		)
-		(stroke
-			(width 0)
-			(type default)
-		)
-	)
-	(wire
-		(pts
 			(xy 91.44 62.23) (xy 91.44 80.01)
 		)
@@
 		)
 		(stroke
-			(width 0)
-			(type default)
-		)
-	)
-	(wire
-		(pts
-			(xy 80.01 107.95) (xy 109.22 107.95)
-		)
-		(stroke
