File: pwm.kicad_sch (KiCad schematic)
At the start: 12 parts, among them IC1 UCC28180D, Q4 T2N7002AK, U10 ICM7555xB, U3 UCC21520DW, U9 CD4053B

Commit message: voltage sense
Parts:
- removed U10: ICM7555xB, Package_SO:SOIC-8_3.9x4.9mm_P1.27mm, symbol Timer:ICM7555xB
Connections:
- net +15V: no longer U3.11 (VDDB)
- net -5V renamed PFC-
- new net PFC+: U3.11 (VDDB)

Commit message: finish initial schematic
Parts:
- added R40: 5.1k 0.1%, Resistor_SMD:R_0805_2012Metric, symbol Device:R
- added R41: 10k 0.1%, Resistor_SMD:R_0805_2012Metric, symbol Device:R
- added R42: 200R, Resistor_SMD:R_0805_2012Metric, symbol Device:R
- added U16: MCP6562, Package_SO:SOIC-8_3.9x4.9mm_P1.27mm, symbol Comparator:MCP6562
- added U17, U18: 74LVC1G02, Package_TO_SOT_SMD:SOT-23-5, symbol 74xGxx:74LVC1G02
- R15: value 5.1k 0.1% -> 5.1k
Connections:
- net +5V: now also R40.2, U16.8 (V+), U17.5 (VCC), U18.5 (VCC)
- net CHARGE_PWM: now also U17.4, U18.1
- net GND: now also R42.1, U16.4 (V-), U17.3 (GND), U18.3 (GND)
- net ISENSE renamed ISENSE_PFC
- new net: U17.2, U18.4
- new net: R41.1, R42.2, U16.3 (+)
- new net: R40.1, R41.2, U16.6 (-)
- new net ISENSE_CHG: U16.2 (-), U16.5 (+)
- new net RESET: U16.7, U17.1
- new net SET: U16.1, U18.2
Other:
- note added: "10A"
- note added: "200mA"
- note added: "320 mV/A"

Commit message: pcb layout
Connections:
- net CHARGE_PWM renamed CHG_PWM

Commit message: pcb work
Parts:
- added C23, C24, C25: 0.1u, Capacitor_SMD:C_0805_2012Metric, symbol Device:C
- added D8: LED_Yellow, LED_SMD:LED_0805_2012Metric, symbol Device:LED
- added D9: LED_Red, LED_SMD:LED_0805_2012Metric, symbol Device:LED
- added R1, R45: 1k, Resistor_SMD:R_0805_2012Metric, symbol Device:R
Connections:
- net +15V: now also C24.1
- net +5V: now also C23.1, C25.1
- net CHARGING: now also R1.1
- net CHSW+: now also U3.11 (VDDB); no longer U3.16 (VDDA)
- net CHSW-: now also U3.9 (VSSB); no longer U3.14 (VSSA)
- net CHSW_GATE: now also U3.10 (OUTB); no longer U3.15 (OUTA)
- net GND: now also C23.2, C24.2, C25.2, D8.1 (K), D9.1 (K)
- net PFC+: now also U3.16 (VDDA); no longer U3.11 (VDDB)
- net PFC-: now also U3.14 (VSSA); no longer U3.9 (VSSB)
- net PFC_GATE: now also U3.15 (OUTA); no longer U3.10 (OUTB)
- net ~{EN}: now also R45.1
- net at U9.14 (A): now also U3.1 (INA); no longer U3.2 (INB)
- net at U9.15 (B): now also U3.2 (INB); no longer U3.1 (INA)
- new net: D9.2 (A), R45.2
- new net: D8.2 (A), R1.2

Commit message: logic layout
Parts:
- added C30: 0.1u, Capacitor_SMD:C_0805_2012Metric, symbol Device:C
Connections:
- net +5V: now also C30.1
- net GND: now also C30.2

Commit message: final touches?
Parts:
- added TP2, TP3: TestPoint, TestPoint:TestPoint_Pad_1.0x1.0mm, symbol Connector:TestPoint
Connections:
- net CHG_PWM: now also TP2.1
- net PFC_PWM: now also TP3.1
Changed lines of the file:
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@@
 	)
 	(junction
+		(at 60.96 107.95)
+		(diameter 0)
+		(color 0 0 0 0)
+	)
+	(junction
 		(at 88.9 111.76)
 		(diameter 0)
@@
 	)
 	(junction
+		(at 63.5 102.87)
+		(diameter 0)
+		(color 0 0 0 0)
+	)
+	(junction
 		(at 170.18 31.75)
 		(diameter 0)
@@
 	(wire
 		(pts
+			(xy 60.96 107.95) (xy 276.86 107.95)
+		)
+		(stroke
+			(width 0)
+			(type default)
+		)
+	)
+	(wire
+		(pts
 			(xy 86.36 111.76) (xy 88.9 111.76)
 		)
@@
 	(wire
 		(pts
-			(xy 157.48 102.87) (xy 54.61 102.87)
+			(xy 157.48 102.87) (xy 63.5 102.87)
 		)
 		(stroke
@@
 	(wire
 		(pts
-			(xy 57.15 107.95) (xy 276.86 107.95)
+			(xy 57.15 107.95) (xy 60.96 107.95)
 		)
 		(stroke
@@
 	(wire
 		(pts
+			(xy 60.96 107.95) (xy 60.96 109.22)
+		)
+		(stroke
+			(width 0)
+			(type default)
+		)
+	)
+	(wire
+		(pts
 			(xy 186.69 66.04) (xy 186.69 67.31)
 		)
@@
 	(wire
 		(pts
+			(xy 63.5 102.87) (xy 63.5 109.22)
+		)
+		(stroke
+			(width 0)
+			(type default)
+		)
+	)
+	(wire
+		(pts
 			(xy 106.68 128.27) (xy 106.68 132.08)
 		)
@@
 	(wire
 		(pts
+			(xy 63.5 102.87) (xy 54.61 102.87)
+		)
+		(stroke
+			(width 0)
+			(type default)
+		)
+	)
+	(wire
+		(pts
 			(xy 222.25 64.77) (xy 226.06 64.77)
 		)
@@
 	)
 	(symbol
+		(lib_id "Connector:TestPoint")
+		(at 60.96 109.22 180)
+		(unit 1)
+		(body_style 1)
+		(exclude_from_sim no)
+		(in_bom yes)
+		(on_board yes)
+		(in_pos_files yes)
+		(dnp no)
+		(fields_autoplaced yes)
+		(property "Reference" "TP2"
+			(at 63.5 111.2519 0)
+			(show_name no)
+			(do_not_autoplace no)
+			(effects
+				(font
+					(size 1.27 1.27)
+				)
+				(justify right)
+			)
+		)
+		(property "Value" "TestPoint"
+			(at 63.5 113.7919 0)
+			(show_name no)
+			(do_not_autoplace no)
+			(effects
+				(font
+					(size 1.27 1.27)
+				)
+				(justify right)
+			)
+		)
+		(property "Footprint" "TestPoint:TestPoint_Pad_1.0x1.0mm"
+			(at 55.88 109.22 0)
+			(hide yes)
+			(show_name no)
+			(do_not_autoplace no)
+			(effects
+				(font
+					(size 1.27 1.27)
+				)
+			)
+		)
+		(property "Datasheet" ""
+			(at 55.88 109.22 0)
+			(hide yes)
+			(show_name no)
+			(do_not_autoplace no)
+			(effects
+				(font
+					(size 1.27 1.27)
+				)
+			)
+		)
+		(property "Description" "test point"
+			(at 60.96 109.22 0)
+			(hide yes)
+			(show_name no)
+			(do_not_autoplace no)
+			(effects
+				(font
+					(size 1.27 1.27)
+				)
+			)
+		)
+		(pin "1"
+		)
+		(instances
+			(project "PFC"
+				(path "/9a4457e8-cc73-4b75-ac20-82cc64952613/9983a37e-d578-4b38-a394-f60aff5d4a98"
+					(reference "TP2")
+					(unit 1)
+				)
+			)
+		)
+	)
+	(symbol
 		(lib_id "power:GND")
 		(at 186.69 87.63 0)
@@
 					(unit 1)
 				)
+			)
+		)
+	)
+	(symbol
+		(lib_id "Connector:TestPoint")
+		(at 63.5 109.22 180)
+		(unit 1)
+		(body_style 1)
+		(exclude_from_sim no)
+		(in_bom yes)
+		(on_board yes)
+		(in_pos_files yes)
+		(dnp no)
+		(fields_autoplaced yes)
+		(property "Reference" "TP3"
+			(at 66.04 111.2519 0)
+			(show_name no)
+			(do_not_autoplace no)
+			(effects
+				(font
+					(size 1.27 1.27)
+				)
+				(justify right)
+			)
+		)
+		(property "Value" "TestPoint"
+			(at 66.04 113.7919 0)
+			(show_name no)
+			(do_not_autoplace no)
+			(effects
+				(font
+					(size 1.27 1.27)
+				)
+				(justify right)
+			)
+		)
+		(property "Footprint" "TestPoint:TestPoint_Pad_1.0x1.0mm"
+			(at 58.42 109.22 0)
+			(hide yes)
+			(show_name no)
+			(do_not_autoplace no)
+			(effects
+				(font
+					(size 1.27 1.27)
+				)
+			)
+		)
+		(property "Datasheet" ""
+			(at 58.42 109.22 0)
+			(hide yes)
+			(show_name no)
+			(do_not_autoplace no)
+			(effects
+				(font
+					(size 1.27 1.27)
+				)
+			)
+		)
+		(property "Description" "test point"
+			(at 63.5 109.22 0)
+			(hide yes)
+			(show_name no)
+			(do_not_autoplace no)
+			(effects
+				(font
+					(size 1.27 1.27)
+				)
+			)
+		)
+		(pin "1"
+		)
+		(instances
+			(project "PFC"
+				(path "/9a4457e8-cc73-4b75-ac20-82cc64952613/9983a37e-d578-4b38-a394-f60aff5d4a98"
+					(reference "TP3")
+					(unit 1)
+				)
